File: pcb/PWM_Bridge_A4955.sch (KiCad schematic (older format))
At the start: 18 parts, among them Q3 IPD220N06L3, Q4 IPD220N06L3, Q5 IPD220N06L3, Q6 IPD220N06L3, U5 A4955GLPTR-T

Commit message: Add more order informations, create BOM
Parts:
- D6, D7, D8, D9: Digi-Key Minimum Quantity (none) -> 1; Digi-Key Part Number (none) -> RB160M-90DKR-ND
- R16: Digi-Key Minimum Quantity (none) -> 1; Digi-Key Part Number (none) -> CRE2512-FZ-R005E-3CT-ND
Changed lines of the file:
@@
 AR Path="/58077727/580787DB" Ref="#PWR063"  Part="1"
 AR Path="/58084D17/580787DB" Ref="#PWR072"  Part="1"
-F 0 "#PWR063" H 5750 5250 50  0001 C CNN
+F 0 "#PWR072" H 5750 5250 50  0001 C CNN
 F 1 "GND" H 5755 5327 50  0000 C CNN
 F 2 "" H 5750 5500 50  0000 C CNN
@@
 AR Path="/58077727/58078835" Ref="#PWR064"  Part="1"
 AR Path="/58084D17/58078835" Ref="#PWR073"  Part="1"
-F 0 "#PWR064" H 4650 5250 50  0001 C CNN
+F 0 "#PWR073" H 4650 5250 50  0001 C CNN
 F 1 "GND" H 4655 5327 50  0000 C CNN
 F 2 "" H 4650 5500 50  0000 C CNN
@@
 F 1 "0R005" H 7670 5105 50  0000 L CNN
 F 2 "Resistors_SMD:R_2512" V 7530 5150 50  0001 C CNN
-F 3 "" H 7600 5150 50  0000 C CNN
+F 3 "http://www.bourns.com/docs/Product-Datasheets/CRE.pdf" H 7600 5150 50  0001 C CNN
+F 4 "CRE2512-FZ-R005E-3CT-ND" H 7600 5150 60  0001 C CNN "Digi-Key Part Number"
+F 5 "1" H 7600 5150 60  0001 C CNN "Digi-Key Minimum Quantity"
 	1    7600 5150
 	1    0    0    -1
@@
 AR Path="/58077727/58078AB1" Ref="#PWR065"  Part="1"
 AR Path="/58084D17/58078AB1" Ref="#PWR074"  Part="1"
-F 0 "#PWR065" H 7600 5250 50  0001 C CNN
+F 0 "#PWR074" H 7600 5250 50  0001 C CNN
 F 1 "GND" H 7605 5327 50  0000 C CNN
 F 2 "" H 7600 5500 50  0000 C CNN
@@
 AR Path="/58077727/5807A4C6" Ref="#PWR066"  Part="1"
 AR Path="/58084D17/5807A4C6" Ref="#PWR075"  Part="1"
-F 0 "#PWR066" H 4950 1900 50  0001 C CNN
+F 0 "#PWR075" H 4950 1900 50  0001 C CNN
 F 1 "GND" H 4955 1977 50  0000 C CNN
 F 2 "" H 4950 2150 50  0000 C CNN
@@
 AR Path="/58077727/5807A964" Ref="#PWR067"  Part="1"
 AR Path="/58084D17/5807A964" Ref="#PWR076"  Part="1"
-F 0 "#PWR067" H 5850 1900 50  0001 C CNN
+F 0 "#PWR076" H 5850 1900 50  0001 C CNN
 F 1 "GND" H 5855 1977 50  0000 C CNN
 F 2 "" H 5850 2150 50  0000 C CNN
@@
 AR Path="/58084D17/5809ACB6" Ref="#PWR077"  Part="1"
 AR Path="/58077727/5809ACB6" Ref="#PWR068"  Part="1"
-F 0 "#PWR068" H 5400 1900 50  0001 C CNN
+F 0 "#PWR077" H 5400 1900 50  0001 C CNN
 F 1 "GND" H 5405 1977 50  0000 C CNN
 F 2 "" H 5400 2150 50  0000 C CNN
@@
 AR Path="/58077727/580A46B3" Ref="#PWR069"  Part="1"
 AR Path="/58084D17/580A46B3" Ref="#PWR078"  Part="1"
-F 0 "#PWR069" H 6300 5250 50  0001 C CNN
+F 0 "#PWR078" H 6300 5250 50  0001 C CNN
 F 1 "GND" H 6305 5327 50  0000 C CNN
 F 2 "" H 6300 5500 50  0000 C CNN
@@
 F 1 "RB160M-60" V 7245 2478 50  0000 L CNN
 F 2 "Diodes_SMD:SOD-123" V 7291 2478 50  0001 L CNN
-F 3 "" H 7200 2400 50  0000 C CNN
+F 3 "http://rohmfs.rohm.com/en/products/databook/datasheet/discrete/diode/schottky_barrier/rb160m-60.pdf" H 7200 2400 50  0001 C CNN
+F 4 "RB160M-90DKR-ND" H 7200 2400 60  0001 C CNN "Digi-Key Part Number"
+F 5 "1" H 7200 2400 60  0001 C CNN "Digi-Key Minimum Quantity"
 	1    7200 2400
 	0    1    1    0
@@
 F 1 "RB160M-60" V 7245 2978 50  0000 L CNN
 F 2 "Diodes_SMD:SOD-123" V 7291 2978 50  0001 L CNN
-F 3 "" H 7200 2900 50  0000 C CNN
+F 3 "http://rohmfs.rohm.com/en/products/databook/datasheet/discrete/diode/schottky_barrier/rb160m-60.pdf" H 7200 2900 50  0001 C CNN
+F 4 "RB160M-90DKR-ND" H 7200 2900 60  0001 C CNN "Digi-Key Part Number"
+F 5 "1" H 7200 2900 60  0001 C CNN "Digi-Key Minimum Quantity"
 	1    7200 2900
 	0    1    1    0
@@
 F 1 "RB160M-60" V 8045 2978 50  0000 L CNN
 F 2 "Diodes_SMD:SOD-123" V 8091 2978 50  0001 L CNN
-F 3 "" H 8000 2900 50  0000 C CNN
+F 3 "http://rohmfs.rohm.com/en/products/databook/datasheet/discrete/diode/schottky_barrier/rb160m-60.pdf" H 8000 2900 50  0001 C CNN
+F 4 "RB160M-90DKR-ND" H 8000 2900 60  0001 C CNN "Digi-Key Part Number"
+F 5 "1" H 8000 2900 60  0001 C CNN "Digi-Key Minimum Quantity"
 	1    8000 2900
 	0    1    1    0
@@
 F 1 "RB160M-60" V 8045 2478 50  0000 L CNN
 F 2 "Diodes_SMD:SOD-123" V 8091 2478 50  0001 L CNN
-F 3 "" H 8000 2400 50  0000 C CNN
+F 3 "http://rohmfs.rohm.com/en/products/databook/datasheet/discrete/diode/schottky_barrier/rb160m-60.pdf" H 8000 2400 50  0001 C CNN
+F 4 "RB160M-90DKR-ND" H 8000 2400 60  0001 C CNN "Digi-Key Part Number"
+F 5 "1" H 8000 2400 60  0001 C CNN "Digi-Key Minimum Quantity"
 	1    8000 2400
 	0    1    1    0
@@
 AR Path="/58077727/581550B7" Ref="#PWR070"  Part="1"
 AR Path="/58084D17/581550B7" Ref="#PWR079"  Part="1"
-F 0 "#PWR070" H 8000 2900 50  0001 C CNN
+F 0 "#PWR079" H 8000 2900 50  0001 C CNN
 F 1 "GND" H 8005 2977 50  0000 C CNN
 F 2 "" H 8000 3150 50  0000 C CNN
@@
 AR Path="/58077727/58155164" Ref="#PWR071"  Part="1"
 AR Path="/58084D17/58155164" Ref="#PWR080"  Part="1"
-F 0 "#PWR071" H 7200 2900 50  0001 C CNN
+F 0 "#PWR080" H 7200 2900 50  0001 C CNN
 F 1 "GND" H 7205 2977 50  0000 C CNN
 F 2 "" H 7200 3150 50  0000 C CNN

Commit message: Add more BOM informations
Parts:
- C17, C18, C19, C20: Digi-Key Minimum Quantity (none) -> 1; Digi-Key Part Number (none) -> 311-1343-1-ND
- C21: Digi-Key Minimum Quantity (none) -> 1; Digi-Key Part Number (none) -> 493-7453-1-ND
- C22: Digi-Key Minimum Quantity (none) -> 1; Digi-Key Part Number (none) -> 311-1081-1-ND
- R14, R15: Digi-Key Minimum Quantity (none) -> 5000; Digi-Key Part Number (none) -> 311-22.0KHRTR-ND
Changed lines of the file:
@@
 F 2 "Capacitors_SMD:C_0603" H 4650 3500 50  0001 C CNN
 F 3 "" H 4650 3500 50  0000 C CNN
+F 4 "311-1343-1-ND" H 4650 3500 60  0001 C CNN "Digi-Key Part Number"
+F 5 "1" H 4650 3500 60  0001 C CNN "Digi-Key Minimum Quantity"
 	1    4650 3500
 	0    1    1    0
@@
 F 2 "Resistors_SMD:R_0603" V 5530 5150 50  0001 C CNN
 F 3 "" H 5600 5150 50  0000 C CNN
+F 4 "311-22.0KHRTR-ND" H 5600 5150 60  0001 C CNN "Digi-Key Part Number"
+F 5 "5000" H 5600 5150 60  0001 C CNN "Digi-Key Minimum Quantity"
 	1    5600 5150
 	1    0    0    -1
@@
 F 2 "Capacitors_SMD:C_0603" H 5938 5000 50  0001 C CNN
 F 3 "" H 5900 5150 50  0000 C CNN
+F 4 "311-1081-1-ND" H 5900 5150 60  0001 C CNN "Digi-Key Part Number"
+F 5 "1" H 5900 5150 60  0001 C CNN "Digi-Key Minimum Quantity"
 	1    5900 5150
 	1    0    0    -1
@@
 AR Path="/58077727/580787DB" Ref="#PWR063"  Part="1"
 AR Path="/58084D17/580787DB" Ref="#PWR072"  Part="1"
-F 0 "#PWR072" H 5750 5250 50  0001 C CNN
+F 0 "#PWR063" H 5750 5250 50  0001 C CNN
 F 1 "GND" H 5755 5327 50  0000 C CNN
 F 2 "" H 5750 5500 50  0000 C CNN
@@
 AR Path="/58077727/58078835" Ref="#PWR064"  Part="1"
 AR Path="/58084D17/58078835" Ref="#PWR073"  Part="1"
-F 0 "#PWR073" H 4650 5250 50  0001 C CNN
+F 0 "#PWR064" H 4650 5250 50  0001 C CNN
 F 1 "GND" H 4655 5327 50  0000 C CNN
 F 2 "" H 4650 5500 50  0000 C CNN
@@
 AR Path="/58077727/58078AB1" Ref="#PWR065"  Part="1"
 AR Path="/58084D17/58078AB1" Ref="#PWR074"  Part="1"
-F 0 "#PWR074" H 7600 5250 50  0001 C CNN
+F 0 "#PWR065" H 7600 5250 50  0001 C CNN
 F 1 "GND" H 7605 5327 50  0000 C CNN
 F 2 "" H 7600 5500 50  0000 C CNN
@@
 F 2 "Capacitors_SMD:C_0603" H 4988 1750 50  0001 C CNN
 F 3 "" H 4950 1900 50  0000 C CNN
+F 4 "311-1343-1-ND" H 4950 1900 60  0001 C CNN "Digi-Key Part Number"
+F 5 "1" H 4950 1900 60  0001 C CNN "Digi-Key Minimum Quantity"
 	1    4950 1900
 	1    0    0    -1
@@
 AR Path="/58077727/5807A4C6" Ref="#PWR066"  Part="1"
 AR Path="/58084D17/5807A4C6" Ref="#PWR075"  Part="1"
-F 0 "#PWR075" H 4950 1900 50  0001 C CNN
+F 0 "#PWR066" H 4950 1900 50  0001 C CNN
 F 1 "GND" H 4955 1977 50  0000 C CNN
 F 2 "" H 4950 2150 50  0000 C CNN
@@
 F 2 "Capacitors_SMD:c_elec_10x10" H 5888 1750 50  0001 C CNN
 F 3 "" H 5850 1900 50  0000 C CNN
+F 4 "493-7453-1-ND" H 5850 1900 60  0001 C CNN "Digi-Key Part Number"
+F 5 "1" H 5850 1900 60  0001 C CNN "Digi-Key Minimum Quantity"
 	1    5850 1900
 	1    0    0    -1
@@
 AR Path="/58077727/5807A964" Ref="#PWR067"  Part="1"
 AR Path="/58084D17/5807A964" Ref="#PWR076"  Part="1"
-F 0 "#PWR076" H 5850 1900 50  0001 C CNN
+F 0 "#PWR067" H 5850 1900 50  0001 C CNN
 F 1 "GND" H 5855 1977 50  0000 C CNN
 F 2 "" H 5850 2150 50  0000 C CNN
@@
 F 2 "Capacitors_SMD:C_0603" H 3700 4850 50  0001 C CNN
 F 3 "" H 3700 4850 50  0000 C CNN
+F 4 "311-1343-1-ND" H 3700 4850 60  0001 C CNN "Digi-Key Part Number"
+F 5 "1" H 3700 4850 60  0001 C CNN "Digi-Key Minimum Quantity"
 	1    3700 4850
 	1    0    0    -1
@@
 F 2 "Capacitors_SMD:C_0603" H 5438 1750 50  0001 C CNN
 F 3 "" H 5400 1900 50  0000 C CNN
+F 4 "311-1343-1-ND" H 5400 1900 60  0001 C CNN "Digi-Key Part Number"
+F 5 "1" H 5400 1900 60  0001 C CNN "Digi-Key Minimum Quantity"
 	1    5400 1900
 	1    0    0    -1
@@
 AR Path="/58084D17/5809ACB6" Ref="#PWR077"  Part="1"
 AR Path="/58077727/5809ACB6" Ref="#PWR068"  Part="1"
-F 0 "#PWR077" H 5400 1900 50  0001 C CNN
+F 0 "#PWR068" H 5400 1900 50  0001 C CNN
 F 1 "GND" H 5405 1977 50  0000 C CNN
 F 2 "" H 5400 2150 50  0000 C CNN
@@
 F 2 "Resistors_SMD:R_0603" V 6230 5150 50  0001 C CNN
 F 3 "" H 6300 5150 50  0000 C CNN
+F 4 "311-22.0KHRTR-ND" H 6300 5150 60  0001 C CNN "Digi-Key Part Number"
+F 5 "5000" H 6300 5150 60  0001 C CNN "Digi-Key Minimum Quantity"
 	1    6300 5150
 	1    0    0    -1
@@
 AR Path="/58077727/580A46B3" Ref="#PWR069"  Part="1"
 AR Path="/58084D17/580A46B3" Ref="#PWR078"  Part="1"
-F 0 "#PWR078" H 6300 5250 50  0001 C CNN
+F 0 "#PWR069" H 6300 5250 50  0001 C CNN
 F 1 "GND" H 6305 5327 50  0000 C CNN
 F 2 "" H 6300 5500 50  0000 C CNN
@@
 AR Path="/58077727/581550B7" Ref="#PWR070"  Part="1"
 AR Path="/58084D17/581550B7" Ref="#PWR079"  Part="1"
-F 0 "#PWR079" H 8000 2900 50  0001 C CNN
+F 0 "#PWR070" H 8000 2900 50  0001 C CNN
 F 1 "GND" H 8005 2977 50  0000 C CNN
 F 2 "" H 8000 3150 50  0000 C CNN
@@
 AR Path="/58077727/58155164" Ref="#PWR071"  Part="1"
 AR Path="/58084D17/58155164" Ref="#PWR080"  Part="1"
-F 0 "#PWR080" H 7200 2900 50  0001 C CNN
+F 0 "#PWR071" H 7200 2900 50  0001 C CNN
 F 1 "GND" H 7205 2977 50  0000 C CNN
 F 2 "" H 7200 3150 50  0000 C CNN

Commit message: Improve BOM
Parts:
- R14, R15: Digi-Key Minimum Quantity 5000 -> 1; Digi-Key Part Number 311-22.0KHRTR-ND -> 311-22.0KHRCT-ND
Changed lines of the file:
@@
 F 2 "Resistors_SMD:R_0603" V 5530 5150 50  0001 C CNN
 F 3 "" H 5600 5150 50  0000 C CNN
-F 4 "311-22.0KHRTR-ND" H 5600 5150 60  0001 C CNN "Digi-Key Part Number"
-F 5 "5000" H 5600 5150 60  0001 C CNN "Digi-Key Minimum Quantity"
+F 4 "311-22.0KHRCT-ND" H 5600 5150 60  0001 C CNN "Digi-Key Part Number"
+F 5 "1" H 5600 5150 60  0001 C CNN "Digi-Key Minimum Quantity"
 	1    5600 5150
 	1    0    0    -1
@@
 AR Path="/58077727/580787DB" Ref="#PWR063"  Part="1"
 AR Path="/58084D17/580787DB" Ref="#PWR072"  Part="1"
-F 0 "#PWR063" H 5750 5250 50  0001 C CNN
+F 0 "#PWR072" H 5750 5250 50  0001 C CNN
 F 1 "GND" H 5755 5327 50  0000 C CNN
 F 2 "" H 5750 5500 50  0000 C CNN
@@
 AR Path="/58077727/58078835" Ref="#PWR064"  Part="1"
 AR Path="/58084D17/58078835" Ref="#PWR073"  Part="1"
-F 0 "#PWR064" H 4650 5250 50  0001 C CNN
+F 0 "#PWR073" H 4650 5250 50  0001 C CNN
 F 1 "GND" H 4655 5327 50  0000 C CNN
 F 2 "" H 4650 5500 50  0000 C CNN
@@
 AR Path="/58077727/58078AB1" Ref="#PWR065"  Part="1"
 AR Path="/58084D17/58078AB1" Ref="#PWR074"  Part="1"
-F 0 "#PWR065" H 7600 5250 50  0001 C CNN
+F 0 "#PWR074" H 7600 5250 50  0001 C CNN
 F 1 "GND" H 7605 5327 50  0000 C CNN
 F 2 "" H 7600 5500 50  0000 C CNN
@@
 AR Path="/58077727/5807A4C6" Ref="#PWR066"  Part="1"
 AR Path="/58084D17/5807A4C6" Ref="#PWR075"  Part="1"
-F 0 "#PWR066" H 4950 1900 50  0001 C CNN
+F 0 "#PWR075" H 4950 1900 50  0001 C CNN
 F 1 "GND" H 4955 1977 50  0000 C CNN
 F 2 "" H 4950 2150 50  0000 C CNN
@@
 AR Path="/58077727/5807A964" Ref="#PWR067"  Part="1"
 AR Path="/58084D17/5807A964" Ref="#PWR076"  Part="1"
-F 0 "#PWR067" H 5850 1900 50  0001 C CNN
+F 0 "#PWR076" H 5850 1900 50  0001 C CNN
 F 1 "GND" H 5855 1977 50  0000 C CNN
 F 2 "" H 5850 2150 50  0000 C CNN
@@
 AR Path="/58084D17/5809ACB6" Ref="#PWR077"  Part="1"
 AR Path="/58077727/5809ACB6" Ref="#PWR068"  Part="1"
-F 0 "#PWR068" H 5400 1900 50  0001 C CNN
+F 0 "#PWR077" H 5400 1900 50  0001 C CNN
 F 1 "GND" H 5405 1977 50  0000 C CNN
 F 2 "" H 5400 2150 50  0000 C CNN
@@
 F 2 "Resistors_SMD:R_0603" V 6230 5150 50  0001 C CNN
 F 3 "" H 6300 5150 50  0000 C CNN
-F 4 "311-22.0KHRTR-ND" H 6300 5150 60  0001 C CNN "Digi-Key Part Number"
-F 5 "5000" H 6300 5150 60  0001 C CNN "Digi-Key Minimum Quantity"
+F 4 "311-22.0KHRCT-ND" H 6300 5150 60  0001 C CNN "Digi-Key Part Number"
+F 5 "1" H 6300 5150 60  0001 C CNN "Digi-Key Minimum Quantity"
 	1    6300 5150
 	1    0    0    -1
@@
 AR Path="/58077727/580A46B3" Ref="#PWR069"  Part="1"
 AR Path="/58084D17/580A46B3" Ref="#PWR078"  Part="1"
-F 0 "#PWR069" H 6300 5250 50  0001 C CNN
+F 0 "#PWR078" H 6300 5250 50  0001 C CNN
 F 1 "GND" H 6305 5327 50  0000 C CNN
 F 2 "" H 6300 5500 50  0000 C CNN
@@
 AR Path="/58077727/581550B7" Ref="#PWR070"  Part="1"
 AR Path="/58084D17/581550B7" Ref="#PWR079"  Part="1"
-F 0 "#PWR070" H 8000 2900 50  0001 C CNN
+F 0 "#PWR079" H 8000 2900 50  0001 C CNN
 F 1 "GND" H 8005 2977 50  0000 C CNN
 F 2 "" H 8000 3150 50  0000 C CNN
@@
 AR Path="/58077727/58155164" Ref="#PWR071"  Part="1"
 AR Path="/58084D17/58155164" Ref="#PWR080"  Part="1"
-F 0 "#PWR071" H 7200 2900 50  0001 C CNN
+F 0 "#PWR080" H 7200 2900 50  0001 C CNN
 F 1 "GND" H 7205 2977 50  0000 C CNN
 F 2 "" H 7200 3150 50  0000 C CNN
