File: pcb/Arduino_Zero_Base.sch (KiCad schematic (older format))
At the start: 14 parts, among them U4 SAMD21G18A-A, Y1 G83270022

Commit message: Add some improvements, fix issue with schematic error
Parts:
- L1: value Ferrite_Bead -> MH1608-471Y
Changed lines of the file:
@@
 LIBS:a4955glptr-t
 LIBS:ap2112k-3.3trg1
+LIBS:lm75bd
+LIBS:mechanical
 LIBS:HighPower-Mechaduino-cache
 EELAYER 25 0
@@
 $EndDescr
 $Comp
-L GND #PWR049
+L GND #PWR053
 U 1 1 5802079F
 P 8800 3350
-F 0 "#PWR049" H 8800 3100 50  0001 C CNN
+F 0 "#PWR053" H 8800 3100 50  0001 C CNN
 F 1 "GND" H 8805 3177 50  0000 C CNN
 F 2 "" H 8800 3350 50  0000 C CNN
@@
 $EndComp
 $Comp
-L GND #PWR050
+L GND #PWR054
 U 1 1 580207D5
 P 9200 3350
-F 0 "#PWR050" H 9200 3100 50  0001 C CNN
+F 0 "#PWR054" H 9200 3100 50  0001 C CNN
 F 1 "GND" H 9205 3177 50  0000 C CNN
 F 2 "" H 9200 3350 50  0000 C CNN
@@
 Connection ~ 8800 2950
 $Comp
-L GND #PWR051
+L GND #PWR055
 U 1 1 58028479
 P 5350 6050
-F 0 "#PWR051" H 5350 5800 50  0001 C CNN
+F 0 "#PWR055" H 5350 5800 50  0001 C CNN
 F 1 "GND" H 5355 5877 50  0000 C CNN
 F 2 "" H 5350 6050 50  0000 C CNN
@@
 $EndComp
 $Comp
-L GND #PWR052
+L GND #PWR056
 U 1 1 5802867C
 P 4950 6050
-F 0 "#PWR052" H 4950 5800 50  0001 C CNN
+F 0 "#PWR056" H 4950 5800 50  0001 C CNN
 F 1 "GND" H 4955 5877 50  0000 C CNN
 F 2 "" H 4950 6050 50  0000 C CNN
@@
 	5250 5950 5250 5850
 $Comp
-L +3V3 #PWR053
+L +3V3 #PWR057
 U 1 1 580289B7
 P 4600 1500
-F 0 "#PWR053" H 4600 1350 50  0001 C CNN
+F 0 "#PWR057" H 4600 1350 50  0001 C CNN
 F 1 "+3V3" H 4615 1673 50  0000 C CNN
 F 2 "" H 4600 1500 50  0000 C CNN
@@
 $EndComp
 $Comp
-L +3V3 #PWR054
+L +3V3 #PWR058
 U 1 1 58028A51
 P 5350 2250
-F 0 "#PWR054" H 5350 2100 50  0001 C CNN
+F 0 "#PWR058" H 5350 2100 50  0001 C CNN
 F 1 "+3V3" H 5365 2423 50  0000 C CNN
 F 2 "" H 5350 2250 50  0000 C CNN
@@
 $EndComp
 $Comp
-L GND #PWR055
+L GND #PWR059
 U 1 1 58028EFC
 P 5550 1950
-F 0 "#PWR055" H 5550 1700 50  0001 C CNN
+F 0 "#PWR059" H 5550 1700 50  0001 C CNN
 F 1 "GND" H 5555 1777 50  0000 C CNN
 F 2 "" H 5550 1950 50  0000 C CNN
@@
 $EndComp
 $Comp
-L GND #PWR056
+L GND #PWR060
 U 1 1 580295A1
 P 4600 2300
-F 0 "#PWR056" H 4600 2050 50  0001 C CNN
+F 0 "#PWR060" H 4600 2050 50  0001 C CNN
 F 1 "GND" H 4605 2127 50  0000 C CNN
 F 2 "" H 4600 2300 50  0000 C CNN
@@
 $EndComp
 $Comp
-L GND #PWR057
+L GND #PWR061
 U 1 1 58029E20
 P 6150 2050
-F 0 "#PWR057" H 6150 1800 50  0001 C CNN
+F 0 "#PWR061" H 6150 1800 50  0001 C CNN
 F 1 "GND" H 6155 1877 50  0000 C CNN
 F 2 "" H 6150 2050 50  0000 C CNN
@@
 $EndComp
 $Comp
-L GND #PWR058
+L GND #PWR062
 U 1 1 58029E5B
 P 7050 2050
-F 0 "#PWR058" H 7050 1800 50  0001 C CNN
+F 0 "#PWR062" H 7050 1800 50  0001 C CNN
 F 1 "GND" H 7055 1877 50  0000 C CNN
 F 2 "" H 7050 2050 50  0000 C CNN
@@
 $EndComp
 $Comp
-L +3V3 #PWR059
+L +3V3 #PWR063
 U 1 1 58029EA6
 P 6150 1650
-F 0 "#PWR059" H 6150 1500 50  0001 C CNN
+F 0 "#PWR063" H 6150 1500 50  0001 C CNN
 F 1 "+3V3" H 6165 1823 50  0000 C CNN
 F 2 "" H 6150 1650 50  0000 C CNN
@@
 $EndComp
 $Comp
-L +3V3 #PWR060
+L +3V3 #PWR064
 U 1 1 58029EE1
 P 7050 1650
-F 0 "#PWR060" H 7050 1500 50  0001 C CNN
+F 0 "#PWR064" H 7050 1500 50  0001 C CNN
 F 1 "+3V3" H 7065 1823 50  0000 C CNN
 F 2 "" H 7050 1650 50  0000 C CNN
@@
 $EndComp
 $Comp
-L +3V3 #PWR061
+L +3V3 #PWR065
 U 1 1 58034CF0
 P 8600 4350
-F 0 "#PWR061" H 8600 4200 50  0001 C CNN
+F 0 "#PWR065" H 8600 4200 50  0001 C CNN
 F 1 "+3V3" H 8615 4523 50  0000 C CNN
 F 2 "" H 8600 4350 50  0000 C CNN
@@
 $EndComp
 $Comp
-L +3V3 #PWR062
+L +3V3 #PWR066
 U 1 1 58034DB6
 P 8900 4350
-F 0 "#PWR062" H 8900 4200 50  0001 C CNN
+F 0 "#PWR066" H 8900 4200 50  0001 C CNN
 F 1 "+3V3" H 8915 4523 50  0000 C CNN
 F 2 "" H 8900 4350 50  0000 C CNN
@@
 $EndComp
 $Comp
-L GND #PWR063
+L GND #PWR067
 U 1 1 5803933E
 P 7550 2250
-F 0 "#PWR063" H 7550 2000 50  0001 C CNN
+F 0 "#PWR067" H 7550 2000 50  0001 C CNN
 F 1 "GND" H 7555 2077 50  0000 C CNN
 F 2 "" H 7550 2250 50  0000 C CNN
@@
 $EndComp
 $Comp
-L GND #PWR064
+L GND #PWR068
 U 1 1 5807F41A
 P 6600 2050
-F 0 "#PWR064" H 6600 1800 50  0001 C CNN
+F 0 "#PWR068" H 6600 1800 50  0001 C CNN
 F 1 "GND" H 6605 1877 50  0000 C CNN
 F 2 "" H 6600 2050 50  0000 C CNN
@@
 $EndComp
 $Comp
-L +3V3 #PWR065
+L +3V3 #PWR069
 U 1 1 5807F420
 P 6600 1650
-F 0 "#PWR065" H 6600 1500 50  0001 C CNN
+F 0 "#PWR069" H 6600 1500 50  0001 C CNN
 F 1 "+3V3" H 6615 1823 50  0000 C CNN
 F 2 "" H 6600 1650 50  0000 C CNN
@@
 P 4600 1750
 F 0 "L1" H 4737 1796 50  0000 L CNN
-F 1 "Ferrite_Bead" H 4737 1705 50  0000 L CNN
+F 1 "MH1608-471Y" H 4737 1705 50  0000 L CNN
 F 2 "Resistors_SMD:R_0603" H 4737 1659 50  0001 L CNN
 F 3 "http://www.bourns.com/docs/Product-Datasheets/mh.pdf" H 4737 1659 50  0001 L CNN
