File: pcb/PoStep25-32_galvanic.sch (KiCad schematic (older format))
At the start: 3 parts, among them P3 PoStep25-32, Q11 BSS138

Commit message: Fix connector footprint
Parts:
- P3: footprint Connectors_Multicomp:Multicomp_MC9A12-1034_2x05x2.54mm_Straight -> Connectors_On-Shore-Technology:On-Shore-Technology_ED1543_2x05x2.54mm_Straight
Changed lines of the file:
@@
 F 0 "P3" H 4650 3265 50  0000 C CNN
 F 1 "PoStep25-32" H 4650 3174 50  0000 C CNN
-F 2 "Connectors_Multicomp:Multicomp_MC9A12-1034_2x05x2.54mm_Straight" H 4650 1650 50  0001 C CNN
+F 2 "Connectors_On-Shore-Technology:On-Shore-Technology_ED1543_2x05x2.54mm_Straight" H 4650 1650 50  0001 C CNN
 F 3 "" H 4650 1650 50  0000 C CNN
 F 4 "ED1543-ND" H 4650 2850 60  0001 C CNN "Digi-Key Part Number"
