File: pcb/Protected_USB_Supply.sch (KiCad schematic (older format))
At the start: 6 parts, among them P2 USB, U7 USBLC6-2SC6

Commit message: Add some improvements, fix issue with schematic error
Parts:
- L2, L3: value Ferrite_Bead -> MH1608-471Y
Changed lines of the file:
@@
 LIBS:a4955glptr-t
 LIBS:ap2112k-3.3trg1
+LIBS:lm75bd
+LIBS:mechanical
 LIBS:HighPower-Mechaduino-cache
 EELAYER 25 0
@@
 	4800 3400 4600 3400
 $Comp
-L GND #PWR086
+L GND #PWR090
 U 1 1 580C177F
 P 4900 4300
-F 0 "#PWR086" H 4900 4050 50  0001 C CNN
+F 0 "#PWR090" H 4900 4050 50  0001 C CNN
 F 1 "GND" H 4905 4127 50  0000 C CNN
 F 2 "" H 4900 4300 50  0000 C CNN
@@
 	4600 3700 4900 3700
 $Comp
-L GND #PWR087
+L GND #PWR091
 U 1 1 580C1786
 P 4200 4400
-F 0 "#PWR087" H 4200 4150 50  0001 C CNN
+F 0 "#PWR091" H 4200 4150 50  0001 C CNN
 F 1 "GND" H 4205 4227 50  0000 C CNN
 F 2 "" H 4200 4400 50  0000 C CNN
@@
 P 6850 2900
 F 0 "L3" V 6576 2900 50  0000 C CNN
-F 1 "Ferrite_Bead" V 6667 2900 50  0000 C CNN
+F 1 "MH1608-471Y" V 6667 2900 50  0000 C CNN
 F 2 "Resistors_SMD:R_0603" V 6668 2900 50  0001 C CNN
 F 3 "http://www.bourns.com/docs/Product-Datasheets/mh.pdf" V 6667 2900 50  0001 C CNN
@@
 P 4200 4150
 F 0 "L2" H 3950 4200 50  0000 L CNN
-F 1 "Ferrite_Bead" H 3550 4100 50  0000 L CNN
+F 1 "MH1608-471Y" H 3550 4100 50  0000 L CNN
 F 2 "Resistors_SMD:R_0603" V 4018 4150 50  0001 C CNN
 F 3 "http://www.bourns.com/docs/Product-Datasheets/mh.pdf" V 4017 4150 50  0001 C CNN
